Commit message: added mesh

File: sock_description/urdf/sock.xacro (robot description, xacro)
@@ -12,8 +12,8 @@
 	<link name="base_link">
 		<visual>
-			<geometry>
-				<box size="${length} ${width} ${height}"/>
-			</geometry>
-			<origin rpy="0 0 0" xyz="0 0 0.032"/>
+      <geometry>
+        <mesh filename="package://sock_description/meshes/sock7.dae"/>
+			</geometry>
+			<origin rpy="0 0 1.57075" xyz="0 0 0.0"/>
 			<material name="color1"/>
 		</visual>
@@ -35,5 +35,5 @@
 		<visual>
 			<geometry>
-				<cylinder length="0.018" radius="0.026"/>
+				<cylinder length="0.001" radius="0.001"/>
 			</geometry>
 			<origin rpy="1.57075 0 0" xyz="0 0.0495 0.0"/>
@@ -57,5 +57,5 @@
 		<visual>
 			<geometry>
-				<cylinder length="0.018" radius="0.026"/>
+				<cylinder length="0.00018" radius="0.00026"/>
 			</geometry>
 			<origin rpy="1.57075 0 0" xyz="0 -0.0495 0.0"/>
@@ -79,5 +79,5 @@
 		<visual>
 			<geometry>
-				<sphere radius="0.026"/>
+				<sphere radius="0.00026"/>
 			</geometry>
 			<origin rpy="0 0 0" xyz="0.0605 0 0.0261"/>
@@ -98,5 +98,5 @@
 		<visual>
 			<geometry>
-				<sphere radius="0.026"/>
+				<sphere radius="0.00026"/>
 			</geometry>
 			<origin rpy="0 0 0" xyz="-0.0605 0 0.0261"/>
